Commit message: Update robot_core.xacro

File: description/robot_core.xacro (robot description, xacro)
@@ -30,4 +30,10 @@
             <material name="white"/>
         </visual>
+        <collision>
+            <origin xyz="0.15 0 0.75"/>
+            <geometry>
+                <box size= "0.3 0.3 0.15"/>
+            </geometry>
+        </collision>
     </link>
     <!-- LEFT WHEEL LNKK-->
@@ -45,4 +51,9 @@
             <material name ="blue"/>
         </visual>
+        <colision>
+            <geometry>
+                 <cylinder radius ="0.05" length="0.04"/>
+            </geometry>
+        </collision>
     </link>
   <!-- right wheel-->
@@ -60,4 +71,9 @@
             <material name ="blue"/>
         </visual>
+        <collision>
+            <geometry>
+                 <cylinder radius ="0.05" length="0.04"/>
+            </geometry>
+        </collision>
     </link>
     <!-- caster wheel joint-->
@@ -72,6 +88,11 @@
                 <sphere radius= "0.05"/>
             </geometry>
+              <material name="black"/>
         </visual>
-        <material name="black"/>
+        <collsion>
+            <geometry>
+                <sphere radius= "0.05"/>
+            </geometry>
+        </collision>
     </link>
 </robot>

Commit message: Update robot_core.xacro

File: description/robot_core.xacro (robot description, xacro)
@@ -37,5 +37,8 @@
             </geometry>
         </collision>
-    </link>
+        <xacro:inertial_box  mass="0.5" x="0.3" y="0.3" z="0.15">
+           <origin xyz ="0.15 0 0.075" rpy="0 0 0"/>
+        </xacro:inertial_box>
+     </link>
     <!-- LEFT WHEEL LNKK-->
     <joint name="left_wheel_joint" type="continuous">
@@ -57,4 +60,7 @@
             </geometry>
         </collision>
+        <xacro:interial_cylinder mass="0.1" radius="0.05" length="0.04">
+            <origin xyz="0 0 0" rpy="0 0 0"/>
+        </xacro:interial_cylinder>
     </link>
   <!-- right wheel-->
@@ -77,4 +83,7 @@
             </geometry>
         </collision>
+        <xacro:inertial_cylinder mass="0.1" radius="0.05" length="0.04">
+            <origin xyz="0 0 0" rpy="0 0 0"/>
+        </xacro:inertial_cylinder>
     </link>
     <!-- caster wheel joint-->
@@ -96,4 +105,7 @@
             </geometry>
         </collision>
+        <xacro:inertial_sphere mass="0.1" radius="0.05">
+            <origin xyz="0 0 0" rpy="0 0 0"/>
+        </xacro:inertial_sphere>
     </link>
 </robot>
